File: fpga_usb/fpga_usb.kicad_pcb (KiCad board)
At the start: 6 copper layers, 38 parts, among them U1 EP2C35F484, U2 FT601Q, U3 FT601Q, U4 AMS1117-3.3, U5 AMS1117-3.3

Commit message: Import USB3 switch. Narrow Netclass.
Parts:
- added C23: 10u, Capacitor_SMD:C_0805_2012Metric, F.Cu at (231.1, 36.7)
- added C24: 10u, Capacitor_SMD:C_0805_2012Metric, F.Cu at (231.1, 15.5)
- added C25: 470n, Capacitor_SMD:C_0603_1608Metric, F.Cu at (215.4, 36.4)
- added C26: 470n, Capacitor_SMD:C_0603_1608Metric, F.Cu at (215.4, 15.3)
- added C27: 470n, Capacitor_SMD:C_0603_1608Metric, F.Cu at (215.4, 39.0)
- added C28: 470n, Capacitor_SMD:C_0603_1608Metric, F.Cu at (215.4, 17.8)
- added C29: 47u, Capacitor_SMD:C_0603_1608Metric, F.Cu at (215.4, 41.5)
- added C30: 47u, Capacitor_SMD:C_0603_1608Metric, F.Cu at (215.4, 20.3)
- added C31: 100n, Capacitor_SMD:C_0201_0603Metric, F.Cu at (230.1, 42.1)
- added C32: 100n, Capacitor_SMD:C_0201_0603Metric, F.Cu at (230.1, 21.0)
- added D2: LED, LED_SMD:LED_0805_2012Metric, F.Cu at (231.1, 39.7)
- added D3: LED, LED_SMD:LED_0805_2012Metric, F.Cu at (231.1, 18.6)
- added J1: Conn_01x02_Pin, Kicad_Personal:TerminalBlock_MAX-MX127-5.0-02P, F.Cu at (220.6, 39.9)
- added J2: Conn_01x02_Pin, Kicad_Personal:TerminalBlock_MAX-MX127-5.0-02P, F.Cu at (220.6, 18.8)
- added JP1: Jumper_3_Open, Connector_PinHeader_2.54mm:PinHeader_1x03_P2.54mm_Vertical, F.Cu at (219.7, 47.0)
- added JP2: Jumper_3_Open, Connector_PinHeader_2.54mm:PinHeader_1x03_P2.54mm_Vertical, F.Cu at (219.7, 25.8)
- added JP3: PWR_MEASURE, Connector_PinHeader_2.54mm:PinHeader_1x02_P2.54mm_Vertical, F.Cu at (229.0, 47.0)
- added JP4: PWR_MEASURE, Connector_PinHeader_2.54mm:PinHeader_1x02_P2.54mm_Vertical, F.Cu at (229.0, 25.8)
- added JP5: Jumper_3_Open, Connector_PinHeader_2.54mm:PinHeader_1x03_P2.54mm_Vertical, F.Cu at (224.3, 47.0)
- added JP6: Jumper_3_Open, Connector_PinHeader_2.54mm:PinHeader_1x03_P2.54mm_Vertical, F.Cu at (224.3, 25.8)
- added R10: 360, Resistor_SMD:R_0603_1608Metric, F.Cu at (215.4, 22.8)
- added R11: 0, Resistor_SMD:R_0603_1608Metric, F.Cu at (215.4, 46.5)
- added R12: 0, Resistor_SMD:R_0603_1608Metric, F.Cu at (215.4, 25.3)
- added R9: 360, Resistor_SMD:R_0603_1608Metric, F.Cu at (215.4, 44.0)
- added U6: PI5USB30213AXEAEX, PI5USB30213AXEAEX-2:QFN40P400X200X50-25N, F.Cu at (164.2, 74.4)
- added U7: PI5USB30213AXEAEX, PI5USB30213AXEAEX-2:QFN40P400X200X50-25N, F.Cu at (164.2, 66.1)
- moved C9 33.7 mm to (172.1, 66.1)
Connections:
- net /F601 USB/5VDC renamed /USB0/5VDC
- net /F601 USB/FT601_GPIO0 renamed /USB0/FT601_GPIO0
- net /F601 USB/FT601_GPIO1 renamed /USB0/FT601_GPIO1
- net /F601 USB/FT601_OE_N renamed /USB0/FT601_OE_N
- net /F601 USB/FT601_RD_N renamed /USB0/FT601_RD_N
- net /F601 USB/FT601_RESET_N renamed /USB0/FT601_RESET_N
- net /F601 USB/FT601_SIWU_N renamed /USB0/FT601_SIWU_N
- net /F601 USB/FT601_WAKEUP_N renamed /USB0/FT601_WAKEUP_N
- net /F601 USB/FT601_WR_N renamed /USB0/FT601_WR_N
- net /F601 USB/RIDN renamed /USB0/RIDN
- net /F601 USB/RIDP renamed /USB0/RIDP
- net /F601 USB/TODN renamed /USB0/TODN
- net /F601 USB/TODP renamed /USB0/TODP
- net /F601 USB/USB_3V3 renamed /USB0/USB_3V3
- net /F601 USB1/5VDC renamed /USB1/5VDC
- net /F601 USB1/FT601_GPIO0 renamed /USB1/FT601_GPIO0
- net /F601 USB1/FT601_GPIO1 renamed /USB1/FT601_GPIO1
- net /F601 USB1/FT601_OE_N renamed /USB1/FT601_OE_N
- net /F601 USB1/FT601_RD_N renamed /USB1/FT601_RD_N
- net /F601 USB1/FT601_RESET_N renamed /USB1/FT601_RESET_N
- net /F601 USB1/FT601_SIWU_N renamed /USB1/FT601_SIWU_N
- net /F601 USB1/FT601_WAKEUP_N renamed /USB1/FT601_WAKEUP_N
- net /F601 USB1/FT601_WR_N renamed /USB1/FT601_WR_N
- net /F601 USB1/RIDN renamed /USB1/RIDN
- net /F601 USB1/RIDP renamed /USB1/RIDP
- net /F601 USB1/TODN renamed /USB1/TODN
- net /F601 USB1/TODP renamed /USB1/TODP
- net /F601 USB1/USB_3V3 renamed /USB1/USB_3V3
- C10 pad 1: unconnected-(C10-Pad1) -> /USB1/TX_P
- C4 pad 1: unconnected-(C4-Pad1) -> /USB0/TX_N
- C5 pad 1: unconnected-(C5-Pad1) -> /USB0/TX_P
- C9 pad 1: unconnected-(C9-Pad1) -> /USB1/TX_N
- U2 pad 37: /F601 USB/VBUS -> /USB0/VBUS
- U3 pad 37: /F601 USB1/VBUS -> /USB1/VBUS
- U4 pad 2: /F601 USB/3V3_LDO -> /USB0/3V3_LDO
- U5 pad 2: /F601 USB1/3V3_LDO -> /USB1/3V3_LDO
Routing:
- net /USB1/TX_N: track 0.00 -> 9.90 mm, vias 0 -> 3
- net /USB1/TODN: track 0.00 -> 4.19 mm, vias 0 -> 1

Commit message: First placement trial of USB0.
Parts:
- removed C1: 4.7u, Capacitor_SMD:C_0603_1608Metric
- removed C2: 470n, Capacitor_SMD:C_0603_1608Metric
- added C33: 100n, Capacitor_SMD:C_0402_1005Metric, F.Cu at (136.0, 142.5)
- added C34: 100n, Capacitor_SMD:C_0402_1005Metric, F.Cu at (136.0, 138.5)
- added C35: 100n, Capacitor_SMD:C_0402_1005Metric, F.Cu at (241.6, 66.7)
- added C36: 100n, Capacitor_SMD:C_0402_1005Metric, F.Cu at (241.6, 69.2)
- added C37: 100n, Capacitor_SMD:C_0402_1005Metric, F.Cu at (136.0, 141.5)
- added C38: 100n, Capacitor_SMD:C_0402_1005Metric, F.Cu at (136.0, 139.5)
- added C39: 100n, Capacitor_SMD:C_0402_1005Metric, F.Cu at (241.6, 71.7)
- added C40: 100n, Capacitor_SMD:C_0402_1005Metric, F.Cu at (241.6, 74.2)
- added C41: 470n, Capacitor_SMD:C_0603_1608Metric, F.Cu at (121.3, 143.0)
- added C42: 470n, Capacitor_SMD:C_0603_1608Metric, F.Cu at (142.2, 109.0)
- added C43: 470n, Capacitor_SMD:C_0603_1608Metric, F.Cu at (121.3, 145.6)
- added C44: 470n, Capacitor_SMD:C_0603_1608Metric, F.Cu at (49.2, 24.5)
- added C45: 470n, Capacitor_SMD:C_0603_1608Metric, F.Cu at (118.8, 150.5)
- added C46: 470n, Capacitor_SMD:C_0603_1608Metric, F.Cu at (130.2, 118.5)
- added C47: 470n, Capacitor_SMD:C_0603_1608Metric, F.Cu at (115.7, 150.5)
- added C48: 470n, Capacitor_SMD:C_0603_1608Metric, F.Cu at (130.2, 121.0)
- added C49: 470n, Capacitor_SMD:C_0603_1608Metric, F.Cu at (121.2, 140.9)
- added C50: 470n, Capacitor_SMD:C_0603_1608Metric, F.Cu at (85.2, 70.7)
- added C51: 3p, Capacitor_SMD:C_0402_1005Metric, F.Cu at (120.1, 147.5)
- added C52: 3p, Capacitor_SMD:C_0402_1005Metric, F.Cu at (0.90, 2.50)
- added J3: USB_C_Receptacle, Connector_USB:USB_C_Receptacle_Amphenol_12401548E4-2A, F.Cu at (149.2, 141.5)
- added J4: USB_C_Receptacle, Connector_USB:USB_C_Receptacle_Amphenol_12401548E4-2A, F.Cu at (233.7, 71.8)
- added R13: 0, Resistor_SMD:R_0402_1005Metric, F.Cu at (126.5, 139.5)
- added R14: 0, Resistor_SMD:R_0402_1005Metric, F.Cu at (241.1, 76.5)
- added R15: 1M, Resistor_SMD:R_0402_1005Metric, F.Cu at (131.5, 137.0)
- added R16: 1M, Resistor_SMD:R_0402_1005Metric, F.Cu at (241.1, 78.4)
- added R17: 0, Resistor_SMD:R_0402_1005Metric, F.Cu at (131.5, 138.0)
- added R18: 0, Resistor_SMD:R_0402_1005Metric, F.Cu at (241.1, 80.4)
- added R19: 0, Resistor_SMD:R_0402_1005Metric, F.Cu at (129.0, 144.6)
- added R20: 0, Resistor_SMD:R_0402_1005Metric, F.Cu at (241.1, 82.4)
- added R21: 0, Resistor_SMD:R_0402_1005Metric, F.Cu at (132.1, 144.6)
- added R22: 0, Resistor_SMD:R_0402_1005Metric, F.Cu at (156.1, 103.7)
- added Y1: X322530MOB4SI, Crystal:Crystal_SMD_3225-4Pin_3.2x2.5mm_HandSoldering, F.Cu at (123.5, 149.1)
- added Y2: X322530MOB4SI, Crystal:Crystal_SMD_3225-4Pin_3.2x2.5mm_HandSoldering, F.Cu at (151.6, 87.2)
- C10, C4, C5, C9: footprint Capacitor_SMD:C_0603_1608Metric -> Capacitor_SMD:C_0402_1005Metric
- C31, C32: footprint Capacitor_SMD:C_0201_0603Metric -> Capacitor_SMD:C_0402_1005Metric
- C6: value 4.7u -> 3p; footprint Capacitor_SMD:C_0603_1608Metric -> Capacitor_SMD:C_0402_1005Metric
- C7: value 470n -> 3p; footprint Capacitor_SMD:C_0603_1608Metric -> Capacitor_SMD:C_0402_1005Metric
- moved C7 213.6 mm to (0.90, 0.53)
- moved D2 164.1 mm to (118.1, 158.7)
- moved C31 159.0 mm to (119.6, 156.5), turned to -90 degrees
- moved JP3 153.7 mm to (122.0, 157.3), turned to 180 degrees
- moved R9 151.6 mm to (118.3, 160.5), turned to 180 degrees
- moved C23 148.2 mm to (140.8, 154.2), turned to 90 degrees
- moved C29 147.9 mm to (119.3, 153.9), turned to 90 degrees
- moved R11 147.2 mm to (121.9, 160.2), turned to 180 degrees
- moved U4 146.9 mm to (132.8, 156.5), turned to 180 degrees
- moved JP5 145.8 mm to (126.2, 154.7)
- moved C27 141.5 mm to (138.4, 157.7), turned to -90 degrees
- moved C25 140.7 mm to (138.4, 154.3), turned to -90 degrees
- moved FB1 138.4 mm to (140.8, 158.5), turned to 90 degrees
- moved J1 138.2 mm to (150.5, 159.0), turned to 90 degrees
- moved JP1 134.6 mm to (144.0, 158.2), turned to 180 degrees
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Connections:
- C11 pad 2: GND -> /USB0/VD10
- C12 pad 2: GND -> /USB1/VD10
- C3 pad 2: GND -> /USB0/VD10
- C6 pad 2: GND -> /USB0/XI
- C7 pad 2: GND -> /USB1/XI
- C8 pad 2: GND -> /USB1/VD10
- R1 pad 1: unconnected-(R1-Pad1) -> /USB0/RX_P
- R1 pad 2: /USB0/RIDN -> /USB0/RIDP
- R2 pad 1: unconnected-(R2-Pad1) -> /USB0/RX_N
- R2 pad 2: /USB0/RIDP -> /USB0/RIDN
- R4 pad 1: unconnected-(R4-Pad1) -> /USB1/RX_P
- R4 pad 2: /USB1/RIDN -> /USB1/RIDP
- R5 pad 1: unconnected-(R5-Pad1) -> /USB1/RX_N
- R5 pad 2: /USB1/RIDP -> /USB1/RIDN
- U2 pad 2: GND -> /USB0/VD10
- U2 pad 21: unconnected-(U2-XI-Pad21) -> /USB0/XI
- U2 pad 22: unconnected-(U2-XO-Pad22) -> /USB0/XO
- U2 pad 23: unconnected-(U2-DP-Pad23) -> /USB0/DP
- U2 pad 25: unconnected-(U2-DM-Pad25) -> /USB0/DM
- U2 pad 3: GND -> /USB0/VD10
- U2 pad 30: GND -> /USB0/VD10
- U2 pad 33: GND -> /USB0/VD10
- U2 pad 34: /USB0/RIDN -> /USB0/RIDP
- U2 pad 35: /USB0/RIDP -> /USB0/RIDN
- U2 pad 39: GND -> /USB0/VD10
- U2 pad 48: GND -> /USB0/VD10
- U3 pad 2: GND -> /USB1/VD10
- U3 pad 21: unconnected-(U3-XI-Pad21) -> /USB1/XI
- U3 pad 22: unconnected-(U3-XO-Pad22) -> /USB1/XO
- U3 pad 23: unconnected-(U3-DP-Pad23) -> /USB1/DP
- U3 pad 25: unconnected-(U3-DM-Pad25) -> /USB1/DM
- U3 pad 3: GND -> /USB1/VD10
- U3 pad 30: GND -> /USB1/VD10
- U3 pad 33: GND -> /USB1/VD10
- U3 pad 34: /USB1/RIDN -> /USB1/RIDP
- U3 pad 35: /USB1/RIDP -> /USB1/RIDN
- U3 pad 39: GND -> /USB1/VD10
- U3 pad 4: /FT601_0_BE0 -> /FT601_1_BE0
- U3 pad 40: /FT601_0_DATA0 -> /FT601_1_DATA0
- U3 pad 41: /FT601_0_DATA1 -> /FT601_1_DATA1
- U3 pad 42: /FT601_0_DATA2 -> /FT601_1_DATA2
- U3 pad 43: /FT601_0_DATA3 -> /FT601_1_DATA3
- U3 pad 44: /FT601_0_DATA4 -> /FT601_1_DATA4
- U3 pad 45: /FT601_0_DATA5 -> /FT601_1_DATA5
- U3 pad 46: /FT601_0_DATA6 -> /FT601_1_DATA6
- U3 pad 47: /FT601_0_DATA7 -> /FT601_1_DATA7
- U3 pad 48: GND -> /USB1/VD10
- U3 pad 5: /FT601_0_BE1 -> /FT601_1_BE1
- U3 pad 50: /FT601_0_DATA8 -> /FT601_1_DATA8
- U3 pad 51: /FT601_0_DATA9 -> /FT601_1_DATA9
- U3 pad 52: /FT601_0_DATA10 -> /FT601_1_DATA10
- U3 pad 53: /FT601_0_DATA11 -> /FT601_1_DATA11
- U3 pad 54: /FT601_0_DATA12 -> /FT601_1_DATA12
- U3 pad 55: /FT601_0_DATA13 -> /FT601_1_DATA13
- U3 pad 56: /FT601_0_DATA14 -> /FT601_1_DATA14
- U3 pad 57: /FT601_0_DATA15 -> /FT601_1_DATA15
- U3 pad 58: /FT601_0_CLK -> /FT601_1_CLK
- U3 pad 6: /FT601_0_BE2 -> /FT601_1_BE2
- U3 pad 60: /FT601_0_DATA16 -> /FT601_1_DATA16
- U3 pad 61: /FT601_0_DATA17 -> /FT601_1_DATA17
- U3 pad 62: /FT601_0_DATA18 -> /FT601_1_DATA18
- U3 pad 63: /FT601_0_DATA19 -> /FT601_1_DATA19
- U3 pad 64: /FT601_0_DATA20 -> /FT601_1_DATA20
- U3 pad 65: /FT601_0_DATA21 -> /FT601_1_DATA21
- U3 pad 66: /FT601_0_DATA22 -> /FT601_1_DATA22
- U3 pad 67: /FT601_0_DATA23 -> /FT601_1_DATA23
- U3 pad 69: /FT601_0_DATA24 -> /FT601_1_DATA24
- U3 pad 7: /FT601_0_BE3 -> /FT601_1_BE3
- U3 pad 70: /FT601_0_DATA25 -> /FT601_1_DATA25
- U3 pad 71: /FT601_0_DATA26 -> /FT601_1_DATA26
- U3 pad 72: /FT601_0_DATA27 -> /FT601_1_DATA27
- U3 pad 73: /FT601_0_DATA28 -> /FT601_1_DATA28
- U3 pad 74: /FT601_0_DATA29 -> /FT601_1_DATA29
- U3 pad 75: /FT601_0_DATA30 -> /FT601_1_DATA30
- U3 pad 76: /FT601_0_DATA31 -> /FT601_1_DATA31
- U3 pad 8: /FT601_0_TXE_N -> /FT601_1_TXE_N
- U3 pad 9: /FT601_0_RXF_N -> /FT601_1_RXF_N
- U6 pad 1: unconnected-(U6-SCL_OUT2-Pad1) -> /USB0/USB_SCL
- U6 pad 10: unconnected-(U6-VCONN-Pad10) -> Net-(U6-VCONN)
- U6 pad 11: unconnected-(U6-CC1-Pad11) -> /USB0/CC1
- U6 pad 12: unconnected-(U6-CC2-Pad12) -> /USB0/CC2
- U6 pad 13: unconnected-(U6-ENB-Pad13) -> Net-(U6-ENB)
- U6 pad 14: unconnected-(U6-B1P-Pad14) -> /USB0/RX1_P
- U6 pad 15: unconnected-(U6-B1N-Pad15) -> /USB0/RX1_N
- U6 pad 16: unconnected-(U6-A1P-Pad16) -> Net-(U6-A1P)
- U6 pad 17: unconnected-(U6-AIN-Pad17) -> Net-(U6-AIN)
- U6 pad 18: unconnected-(U6-B2N-Pad18) -> /USB0/RX2_N
- U6 pad 19: unconnected-(U6-B2P-Pad19) -> /USB0/RX2_P
- U6 pad 2: unconnected-(U6-INTB_OUT3-Pad2) -> /USB0/USB_INTB
- U6 pad 20: unconnected-(U6-A2N-Pad20) -> Net-(U6-A2N)
- U6 pad 21: unconnected-(U6-A2P-Pad21) -> Net-(U6-A2P)
- U6 pad 22: unconnected-(U6-ADDR-Pad22) -> Net-(U6-ADDR)
- U6 pad 23: unconnected-(U6-VBUSDET-Pad23) -> Net-(U6-VBUSDET)
- U6 pad 24: unconnected-(U6-SDA_OUT1-Pad24) -> /USB0/USB_SDA
- U6 pad 25: unconnected-(U6-GND-Pad25) -> GND
- U6 pad 3: unconnected-(U6-PORT-Pad3) -> Net-(U6-PORT)
- U6 pad 6: unconnected-(U6-VDD-Pad6) -> /USB0/USB_3V3
- U6 pad 7: unconnected-(U6-BN-Pad7) -> /USB0/RX_N
- U6 pad 8: unconnected-(U6-BP-Pad8) -> /USB0/RX_P
- U6 pad 9: unconnected-(U6-ID-Pad9) -> /USB0/USB_ID
- U7 pad 1: unconnected-(U7-SCL_OUT2-Pad1) -> /USB1/USB_SCL
- U7 pad 10: unconnected-(U7-VCONN-Pad10) -> Net-(U7-VCONN)
- U7 pad 11: unconnected-(U7-CC1-Pad11) -> /USB1/CC1
- U7 pad 12: unconnected-(U7-CC2-Pad12) -> /USB1/CC2
- U7 pad 13: unconnected-(U7-ENB-Pad13) -> Net-(U7-ENB)
- U7 pad 14: unconnected-(U7-B1P-Pad14) -> /USB1/RX1_P
- U7 pad 15: unconnected-(U7-B1N-Pad15) -> /USB1/RX1_N
- U7 pad 16: unconnected-(U7-A1P-Pad16) -> Net-(U7-A1P)
- U7 pad 17: unconnected-(U7-AIN-Pad17) -> Net-(U7-AIN)
- U7 pad 18: unconnected-(U7-B2N-Pad18) -> /USB1/RX2_N
- U7 pad 19: unconnected-(U7-B2P-Pad19) -> /USB1/RX2_P
- U7 pad 2: unconnected-(U7-INTB_OUT3-Pad2) -> /USB1/USB_INTB
- U7 pad 20: unconnected-(U7-A2N-Pad20) -> Net-(U7-A2N)
- U7 pad 21: unconnected-(U7-A2P-Pad21) -> Net-(U7-A2P)
- U7 pad 22: unconnected-(U7-ADDR-Pad22) -> Net-(U7-ADDR)
- U7 pad 23: unconnected-(U7-VBUSDET-Pad23) -> Net-(U7-VBUSDET)
- U7 pad 24: unconnected-(U7-SDA_OUT1-Pad24) -> /USB1/USB_SDA
- U7 pad 25: unconnected-(U7-GND-Pad25) -> GND
- U7 pad 3: unconnected-(U7-PORT-Pad3) -> Net-(U7-PORT)
- U7 pad 6: unconnected-(U7-VDD-Pad6) -> /USB1/USB_3V3
- U7 pad 7: unconnected-(U7-BN-Pad7) -> /USB1/RX_N
- U7 pad 8: unconnected-(U7-BP-Pad8) -> /USB1/RX_P
- U7 pad 9: unconnected-(U7-ID-Pad9) -> /USB1/USB_ID
Routing:
- net /USB0/DM: track 0.00 -> 29.3 mm, vias 0 -> 2
- net /USB0/DP: track 0.00 -> 28.9 mm, vias 0 -> 3
- net /USB0/CC2: track 0.00 -> 23.3 mm, vias 0 -> 1
- net /USB0/USB_3V3: track 0.00 -> 22.4 mm, vias 0 -> 3
- net /USB0/RX1_P: track 0.00 -> 15.2 mm, vias 0 -> 1
- net /USB0/RX1_N: track 0.00 -> 15.2 mm, vias 0 -> 1
- net /USB0/RX2_P: track 0.00 -> 13.3 mm
- net /USB0/RX2_N: track 0.00 -> 13.2 mm
- net /USB0/VBUS: track 0.00 -> 12.2 mm, vias 0 -> 3
- net /USB0/TX2_N: track 0.00 -> 10.2 mm, vias 0 -> 1
- net /USB0/TX2_P: track 0.00 -> 10.0 mm, vias 0 -> 1
- net /USB0/RIDP: track 0.00 -> 9.03 mm, vias 0 -> 2
- net /USB0/TX1_P: track 0.00 -> 8.77 mm
- net /USB0/FT601_WR_N: track 0.00 -> 8.75 mm, vias 0 -> 1
- net /USB0/RIDN: track 0.00 -> 8.70 mm, vias 0 -> 2
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